File: 2_hardware/1_ArduinoShields/FotoMindARShield.sch (EAGLE design)
At the start: 0 parts

Commit message: Editing Shield & Adding optocouplers
Parts:
- added OK1, OK2, OK3: 4N35, optocoupler:4N35
- added PCB1: ARDUINO_UNO, E14_Arduino_published:ARDUINO_UNO
- added R1, R2, R3: 1k, eagle-ltspice:R0204/7
Connections:
- new net GND: OK1.C, OK2.C, OK3.C
- new net N$1: OK1.A, R1.1
- new net N$2: OK2.A, R2.1
- new net N$3: OK3.A, R3.1
- new net N$4: PCB1.8, R1.2
- new net N$5: PCB1.~10, R2.2
- new net N$6: PCB1.~9, R3.2
Changed lines of the file:
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@@
 <layer number="97" name="Info" color="7" fill="1" visible="yes" active="yes"/>
 <layer number="98" name="Guide" color="6" fill="1" visible="yes" active="yes"/>
+<layer number="99" name="SpiceOrder" color="5" fill="1" visible="yes" active="yes"/>
 <layer number="100" name="Muster" color="7" fill="1" visible="no" active="no"/>
 <layer number="101" name="Patch_Top" color="12" fill="4" visible="yes" active="yes"/>
@@
 </classes>
 <parts>
+<part name="PCB1" library="E14_Arduino_published" deviceset="ARDUINO_UNO" device=""/>
+<part name="OK1" library="optocoupler" deviceset="4N35" device=""/>
+<part name="OK2" library="optocoupler" deviceset="4N35" device=""/>
+<part name="OK3" library="optocoupler" deviceset="4N35" device=""/>
+<part name="R1" library="eagle-ltspice" deviceset="R" device="0204/7" value="1k"/>
+<part name="R2" library="eagle-ltspice" deviceset="R" device="0204/7" value="1k"/>
+<part name="R3" library="eagle-ltspice" deviceset="R" device="0204/7" value="1k"/>
+<part name="GND1" library="supply1" deviceset="GND" device=""/>
+<part name="GND2" library="supply1" deviceset="GND" device=""/>
+<part name="GND3" library="supply1" deviceset="GND" device=""/>
 </parts>
 <sheets>
@@
 </plain>
 <instances>
+<instance part="PCB1" gate="G$1" x="88.9" y="48.26" rot="R90"/>
+<instance part="OK1" gate="G$1" x="17.78" y="66.04" rot="R180"/>
+<instance part="OK2" gate="G$1" x="17.78" y="48.26" rot="R180"/>
+<instance part="OK3" gate="G$1" x="17.78" y="30.48" rot="R180"/>
+<instance part="R1" gate="G$1" x="38.1" y="63.5"/>
+<instance part="R2" gate="G$1" x="38.1" y="45.72"/>
+<instance part="R3" gate="G$1" x="38.1" y="27.94"/>
+<instance part="GND1" gate="1" x="30.48" y="68.58"/>
+<instance part="GND2" gate="1" x="30.48" y="50.8"/>
+<instance part="GND3" gate="1" x="30.48" y="33.02"/>
 </instances>
 <busses>
 </busses>
 <nets>
+<net name="GND" class="0">
+<segment>
+<pinref part="OK1" gate="G$1" pin="C"/>
+<pinref part="GND1" gate="1" pin="GND"/>
+<wire x1="27.94" y1="71.12" x2="30.48" y2="71.12" width="0.1524" layer="91"/>
+</segment>
+<segment>
+<pinref part="OK2" gate="G$1" pin="C"/>
+<pinref part="GND2" gate="1" pin="GND"/>
+<wire x1="27.94" y1="53.34" x2="30.48" y2="53.34" width="0.1524" layer="91"/>
+</segment>
+<segment>
+<pinref part="OK3" gate="G$1" pin="C"/>
+<pinref part="GND3" gate="1" pin="GND"/>
+<wire x1="27.94" y1="35.56" x2="30.48" y2="35.56" width="0.1524" layer="91"/>
+</segment>
+</net>
+<net name="N$1" class="0">
+<segment>
+<pinref part="OK1" gate="G$1" pin="A"/>
+<pinref part="R1" gate="G$1" pin="1"/>
+<wire x1="27.94" y1="63.5" x2="33.02" y2="63.5" width="0.1524" layer="91"/>
+</segment>
+</net>
+<net name="N$2" class="0">
+<segment>
+<pinref part="OK2" gate="G$1" pin="A"/>
+<pinref part="R2" gate="G$1" pin="1"/>
+<wire x1="27.94" y1="45.72" x2="33.02" y2="45.72" width="0.1524" layer="91"/>
+</segment>
+</net>
+<net name="N$3" class="0">
+<segment>
+<pinref part="OK3" gate="G$1" pin="A"/>
+<pinref part="R3" gate="G$1" pin="1"/>
+<wire x1="27.94" y1="27.94" x2="33.02" y2="27.94" width="0.1524" layer="91"/>
+</segment>
+</net>
+<net name="N$4" class="0">
+<segment>
+<pinref part="PCB1" gate="G$1" pin="8"/>
+<wire x1="68.58" y1="48.26" x2="55.88" y2="48.26" width="0.1524" layer="91"/>
+<wire x1="55.88" y1="48.26" x2="55.88" y2="63.5" width="0.1524" layer="91"/>
+<wire x1="55.88" y1="63.5" x2="43.18" y2="63.5" width="0.1524" layer="91"/>
+<pinref part="R1" gate="G$1" pin="2"/>
+</segment>
+</net>
+<net name="N$5" class="0">
+<segment>
+<pinref part="PCB1" gate="G$1" pin="~10"/>
+<wire x1="68.58" y1="43.18" x2="45.72" y2="43.18" width="0.1524" layer="91"/>
+<wire x1="45.72" y1="43.18" x2="45.72" y2="45.72" width="0.1524" layer="91"/>
+<pinref part="R2" gate="G$1" pin="2"/>
+<wire x1="45.72" y1="45.72" x2="43.18" y2="45.72" width="0.1524" layer="91"/>
+</segment>
+</net>
+<net name="N$6" class="0">
+<segment>
+<pinref part="R3" gate="G$1" pin="2"/>
+<wire x1="43.18" y1="27.94" x2="55.88" y2="27.94" width="0.1524" layer="91"/>
+<wire x1="55.88" y1="27.94" x2="55.88" y2="45.72" width="0.1524" layer="91"/>
+<pinref part="PCB1" gate="G$1" pin="~9"/>
+<wire x1="55.88" y1="45.72" x2="68.58" y2="45.72" width="0.1524" layer="91"/>
+</segment>
+</net>
 </nets>
 </sheet>
